File: schematic/12.지그보드 커넥터 배치도(KiCad)_v1.1/콘솔형/AMDS_콘솔형 지그보드_1.1A_커넥터 배치도.kicad_sch (KiCad schematic)
At the start: 43 parts, among them J1 Fan1, J1C03 TEMP, J1C04 LED_DP1, J1C05 LED_DP2, J1C06 LED_TEMP, J1C07 LED_PSU, J1C08 LED_FAN#1, J1C09 LED_FAN#2, J1C1 POWER, J1C10 DP_USB_SW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

Commit message: 24.12.21C
Parts:
- removed D3: TEMP, symbol Device:LED_RKBG
- removed D4: PSU, symbol Device:LED_RKBG
- removed D5: FAN#1, symbol Device:LED_RKBG
- removed D6: FAN#2, symbol Device:LED_RKBG
- removed J1C2: FAN, symbol Connector_Generic:Conn_02x10_Top_Bottom
- added D3: TEMP, symbol Device:LED_RKGB
- added D4: PSU, symbol Device:LED_RKGB
- added D5: FAN#1, symbol Device:LED_RKGB
- added D6: FAN#2, symbol Device:LED_RKGB
- added J10: TEMP2, symbol Connector:Conn_01x04_Socket
- added J7, J8: Conn_01x10, symbol Connector_Generic:Conn_01x10
- added J9: TEMP1, symbol Connector:Conn_01x04_Socket
- J1C03: value TEMP -> TEMP#
- renumbered D7 to D2
Connections:
- net PWM_FAN#3 is gone; now on net PWM_FAN#2: J5.1 (Pin_1), J6.1 (Pin_1)
- net +24V: now also J7.1 (Pin_1), J7.2 (Pin_2), J8.1 (Pin_1), J8.2 (Pin_2)
- net +5V: no longer TEMP1.1 (Vdd), TEMP2.1 (Vdd)
- net GND: now also D3.2 (K), D4.2 (K), D5.2 (K), D6.2 (K), J10.2 (Pin_2), J9.2 (Pin_2)
- net GND2: now also J7.3 (Pin_3), J7.4 (Pin_4), J8.3 (Pin_3), J8.4 (Pin_4)
- net LED_FAN1_G: now also D5.3 (GA)
- net LED_FAN1_R: now also J1C08.3 (Pin_3), D5.1 (RA)
- net LED_FAN2_G: now also D6.3 (GA)
- net LED_FAN2_R: now also J1C09.3 (Pin_3), D6.1 (RA)
- net LED_PSU_G: now also D4.3 (GA)
- net LED_PSU_R: now also J1C07.3 (Pin_3), D4.1 (RA)
- net LED_TEMP_G: now also D3.3 (GA)
- net LED_TEMP_R: now also D3.1 (RA)
- net SCL1: now also J9.3 (Pin_3)
- net SCL2: now also J10.3 (Pin_3)
- net SDA1: now also J9.4 (Pin_4)
- net SDA2: now also J10.4 (Pin_4)
- net SEL_DP1: now also J1C10.1 (Pin_1); no longer J1C10.3 (Pin_3)
- net SEL_DP2: now also J1C10.3 (Pin_3); no longer J1C10.1 (Pin_1)
- new net VDD: J10.1 (Pin_1), J9.1 (Pin_1), TEMP1.1 (Vdd), TEMP2.1 (Vdd)
Other:
- note added: "콘솔형 지그보드 핀맵"
- note removed: "콘솔형 지그보드"
- moved on the sheet: D1, D2, FAN1, J1, J1C03, J1C04, J1C05, J1C06, J1C07, J1C08, J1C09, J1C1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
